File: hardware/pcb/FolkraceCar2020.sch (KiCad schematic (older format))
At the start: 73 parts, among them IC1 DRV8874PWPR, J1 Conn_01x02_Male, J2 Raspberry_Pi, J3 Conn_01x02_Male, J4 Conn Servo, J5 Conn Fan, J6 Conn Hall Effect, J7 Conn_01x06_Male, J8 Conn_01x06_Male, J9 Conn_01x06_Male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

Commit message: Finished with rev 1
Parts:
- added R26: R, Resistor_SMD:R_0603_1608Metric, symbol Device:R
Connections:
- net B1: now also J2.7 (GCLK0/GPIO4)
- net B2: now also J2.11 (GPIO17)
- net FAN_CTRL: now also J2.15 (GPIO22)
- net Start: now also J2.13 (GPIO27)
- net ~SHDN_TOF_1: now also J2.16 (GPIO23)
- net ~SHDN_TOF_2: now also J2.12 (GPIO18/PWM0)
- net ~SHDN_TOF_3: now also J2.29 (GCLK1/GPIO5)
- net PGOOD: now reaches Q1.1 (G), R17.1, U2.2 (PGOOD)
- net PGOOD: now also R26.2
- net NSLEEP: now reaches IC1.3 (NSLEEP), R13.1
- net NSLEEP: now also R26.1
- net ~PGOOD: now reaches Q1.3 (D), R19.2
- no-connect marks 9 -> 11
Other:
- note removed: "ADD BULK CAP!!!"
- moved on the sheet: D1, R13, R8
Changed lines of the file:
@@
 L Device:LED D1
 U 1 1 5EA6C68B
-P 5750 9100
-F 0 "D1" H 5743 9316 50  0000 C CNN
-F 1 "LED RED" H 5743 9225 50  0000 C CNN
-F 2 "LED_SMD:LED_0603_1608Metric" H 5750 9100 50  0001 C CNN
-F 3 "~" H 5750 9100 50  0001 C CNN
-	1    5750 9100
+P 5500 9100
+F 0 "D1" H 5493 9316 50  0000 C CNN
+F 1 "LED RED" H 5493 9225 50  0000 C CNN
+F 2 "LED_SMD:LED_0603_1608Metric" H 5500 9100 50  0001 C CNN
+F 3 "~" H 5500 9100 50  0001 C CNN
+	1    5500 9100
 	0    -1   -1   0
 $EndComp
@@
 L Device:R R8
 U 1 1 5EA6E3FF
-P 5750 8700
-F 0 "R8" H 5650 8800 50  0000 C CNN
-F 1 "R" H 5634 8700 50  0000 C CNN
-F 2 "Resistor_SMD:R_0603_1608Metric" V 5680 8700 50  0001 C CNN
-F 3 "~" H 5750 8700 50  0001 C CNN
-	1    5750 8700
-	1    0    0    -1
-$EndComp
-Wire Wire Line
-	5750 9350 6600 9350
+P 5500 8700
+F 0 "R8" H 5400 8800 50  0000 C CNN
+F 1 "R" H 5384 8700 50  0000 C CNN
+F 2 "Resistor_SMD:R_0603_1608Metric" V 5430 8700 50  0001 C CNN
+F 3 "~" H 5500 8700 50  0001 C CNN
+	1    5500 8700
+	1    0    0    -1
+$EndComp
+Wire Wire Line
+	5500 9350 6600 9350
 $Comp
 L power:+5V #PWR012
 U 1 1 5EA7FCA3
-P 5750 8350
-F 0 "#PWR012" H 5750 8200 50  0001 C CNN
-F 1 "+5V" H 5765 8523 50  0000 C CNN
-F 2 "" H 5750 8350 50  0001 C CNN
-F 3 "" H 5750 8350 50  0001 C CNN
-	1    5750 8350
-	1    0    0    -1
-$EndComp
-Wire Wire Line
-	5750 8350 5750 8450
+P 5500 8350
+F 0 "#PWR012" H 5500 8200 50  0001 C CNN
+F 1 "+5V" H 5515 8523 50  0000 C CNN
+F 2 "" H 5500 8350 50  0001 C CNN
+F 3 "" H 5500 8350 50  0001 C CNN
+	1    5500 8350
+	1    0    0    -1
+$EndComp
+Wire Wire Line
+	5500 8350 5500 8450
 Wire Wire Line
 	3550 9800 3750 9800
@@
 SCL
 Wire Wire Line
-	3150 5550 3350 5550
-Wire Wire Line
-	3150 5450 3350 5450
-Text Label 3350 5550 2    50   ~ 0
+	3150 5550 3650 5550
+Wire Wire Line
+	3150 5450 3650 5450
+Text Label 3650 5550 2    50   ~ 0
 SCL
-Text Label 3350 5450 2    50   ~ 0
+Text Label 3650 5450 2    50   ~ 0
 SDA
-Text Notes 8000 10050 0    50   ~ 0
-ADD BULK CAP!!!
-$Comp
-L Device:R R13
-U 1 1 5EAAF207
-P 6150 8700
-F 0 "R13" H 6220 8746 50  0000 L CNN
-F 1 "R" H 6220 8655 50  0000 L CNN
-F 2 "Resistor_SMD:R_0603_1608Metric" V 6080 8700 50  0001 C CNN
-F 3 "~" H 6150 8700 50  0001 C CNN
-	1    6150 8700
-	-1   0    0    1
-$EndComp
-Connection ~ 5750 8450
-Wire Wire Line
-	5750 8450 5750 8550
-Wire Wire Line
-	6150 8550 6150 8450
-Wire Wire Line
-	6150 8850 6150 9250
-Wire Wire Line
-	6150 9250 6600 9250
-Wire Wire Line
-	5750 8450 6150 8450
+Connection ~ 5500 8450
+Wire Wire Line
+	5500 8450 5500 8550
+Wire Wire Line
+	5900 9250 6200 9250
+Wire Wire Line
+	5500 8450 5900 8450
 $Comp
 L Device:R R18
@@
 $EndComp
 Wire Wire Line
-	5750 8850 5750 8950
-Wire Wire Line
-	5750 9250 5750 9350
+	5500 8850 5500 8950
+Wire Wire Line
+	5500 9250 5500 9350
 Text Notes 6800 8100 0    50   ~ 0
 Motor Driver\nPMODE = 0 -> PH/EN Control mode\nnSLEEP = 1 -> Sleep disabled
@@
 Text Notes 5400 9750 3    50   ~ 0
 Deglitch cap
-Text Label 3450 6750 2    50   ~ 0
+Text Label 3650 6750 2    50   ~ 0
 PWM_M
-Text Label 3400 5950 2    50   ~ 0
+Text Label 3650 5950 2    50   ~ 0
 DIR_M
 Wire Wire Line
-	3150 5950 3400 5950
-Wire Wire Line
-	3150 6750 3450 6750
+	3150 5950 3650 5950
+Wire Wire Line
+	3150 6750 3650 6750
 $Comp
 L power:GND #PWR019
@@
 NoConn ~ 1550 5150
 NoConn ~ 1550 5250
+Text Label 3650 5750 2    50   ~ 0
+B1
+Wire Wire Line
+	3150 5750 3650 5750
+Text Label 1050 5550 0    50   ~ 0
+B2
+Wire Wire Line
+	1550 5550 1050 5550
+Text Label 1050 5650 0    50   ~ 0
+~SHDN_TOF_2
+Wire Wire Line
+	1550 5650 1050 5650
+Text Label 3650 5850 2    50   ~ 0
+~SHDN_TOF_3
+NoConn ~ 3150 5150
+NoConn ~ 3150 5250
+Wire Wire Line
+	3150 5850 3650 5850
+Text Label 7800 1700 0    50   ~ 0
+~PGOOD
+Text Label 6350 9250 0    50   ~ 0
+NSLEEP
+Wire Wire Line
+	5900 8550 5900 8450
+Wire Wire Line
+	5900 8850 5900 9250
+$Comp
+L Device:R R13
+U 1 1 5EAAF207
+P 5900 8700
+F 0 "R13" H 5970 8746 50  0000 L CNN
+F 1 "R" H 5970 8655 50  0000 L CNN
+F 2 "Resistor_SMD:R_0603_1608Metric" V 5830 8700 50  0001 C CNN
+F 3 "~" H 5900 8700 50  0001 C CNN
+	1    5900 8700
+	-1   0    0    1
+$EndComp
+$Comp
+L Device:R R26
+U 1 1 5E9F596A
+P 6200 8700
+F 0 "R26" H 6270 8746 50  0000 L CNN
+F 1 "R" H 6270 8655 50  0000 L CNN
+F 2 "Resistor_SMD:R_0603_1608Metric" V 6130 8700 50  0001 C CNN
+F 3 "~" H 6200 8700 50  0001 C CNN
+	1    6200 8700
+	-1   0    0    1
+$EndComp
+Wire Wire Line
+	6200 8850 6200 9250
+Connection ~ 6200 9250
+Wire Wire Line
+	6200 9250 6600 9250
+Text Label 5900 2650 0    50   ~ 0
+PGOOD
+Wire Wire Line
+	6200 8550 6200 8450
+Wire Wire Line
+	6200 8450 6700 8450
+Text Label 6700 8450 2    50   ~ 0
+PGOOD
+Text Label 1050 6750 0    50   ~ 0
+Start
+Wire Wire Line
+	1050 6750 1550 6750
+Text Label 1050 6250 0    50   ~ 0
+FAN_CTRL
+Wire Wire Line
+	1050 6250 1550 6250
+Text Label 1050 6350 0    50   ~ 0
+~SHDN_TOF_1
+Wire Wire Line
+	1050 6350 1550 6350
 $EndSCHEMATC

Commit message: fixed 3v3 error
Connections:
- net +5V: no longer C2.1, J6.4 (Pin_4), R10.1, R11.1, R23.1, R25.1, U1.8 (VDD)
- net ME_A: now also J2.18 (GPIO24)
- net ME_B: now also J2.22 (GPIO25)
- net +3V3: now reaches J2.1 (3V3)
- net +3V3: now also C2.1, J2.17 (3V3), J6.4 (Pin_4), R10.1, R11.1, R23.1, R25.1, U1.8 (VDD)
- no-connect marks 11 -> 9
Changed lines of the file:
@@
 	-1   0    0    1
-$EndComp
-$Comp
-L power:+5V #PWR031
-U 1 1 5EDCE584
-P 12050 6650
-F 0 "#PWR031" H 12050 6500 50  0001 C CNN
-F 1 "+5V" H 11900 6700 50  0000 C CNN
-F 2 "" H 12050 6650 50  0001 C CNN
-F 3 "" H 12050 6650 50  0001 C CNN
-	1    12050 6650
-	1    0    0    -1
 $EndComp
 Wire Wire Line
@@
 Text Label 12050 4650 0    50   ~ 0
 FAN-
-$Comp
-L power:+5V #PWR07
-U 1 1 5EB6286D
-P 3150 8600
-F 0 "#PWR07" H 3150 8450 50  0001 C CNN
-F 1 "+5V" H 3165 8773 50  0000 C CNN
-F 2 "" H 3150 8600 50  0001 C CNN
-F 3 "" H 3150 8600 50  0001 C CNN
-	1    3150 8600
-	1    0    0    -1
-$EndComp
 Text Notes 2300 10350 0    50   ~ 0
 I2C Adress:\nGND -> 1001000\n
@@
 	1    0    0    -1
 $EndComp
-NoConn ~ 2550 4750
-NoConn ~ 2450 4750
 $Comp
 L Device:R R11
@@
 	1    6000 6050
 	0    1    1    0
-$EndComp
-$Comp
-L power:+5V #PWR014
-U 1 1 5F15381D
-P 6350 5800
-F 0 "#PWR014" H 6350 5650 50  0001 C CNN
-F 1 "+5V" H 6365 5973 50  0000 C CNN
-F 2 "" H 6350 5800 50  0001 C CNN
-F 3 "" H 6350 5800 50  0001 C CNN
-	1    6350 5800
-	1    0    0    -1
 $EndComp
 Wire Wire Line
@@
 Wire Wire Line
 	1050 6350 1550 6350
+$Comp
+L power:+3.3V #PWR0101
+U 1 1 5E843369
+P 2450 4550
+F 0 "#PWR0101" H 2450 4400 50  0001 C CNN
+F 1 "+3.3V" H 2465 4723 50  0000 C CNN
+F 2 "" H 2450 4550 50  0001 C CNN
+F 3 "" H 2450 4550 50  0001 C CNN
+	1    2450 4550
+	1    0    0    -1
+$EndComp
+Wire Wire Line
+	2450 4550 2450 4650
+Wire Wire Line
+	2450 4650 2550 4650
+Wire Wire Line
+	2550 4650 2550 4750
+Connection ~ 2450 4650
+Wire Wire Line
+	2450 4650 2450 4750
+$Comp
+L power:+3.3V #PWR0102
+U 1 1 5E87B61B
+P 6350 5800
+F 0 "#PWR0102" H 6350 5650 50  0001 C CNN
+F 1 "+3.3V" H 6365 5973 50  0000 C CNN
+F 2 "" H 6350 5800 50  0001 C CNN
+F 3 "" H 6350 5800 50  0001 C CNN
+	1    6350 5800
+	1    0    0    -1
+$EndComp
+$Comp
+L power:+3.3V #PWR0103
+U 1 1 5E87D24A
+P 12050 6650
+F 0 "#PWR0103" H 12050 6500 50  0001 C CNN
+F 1 "+3.3V" H 12065 6823 50  0000 C CNN
+F 2 "" H 12050 6650 50  0001 C CNN
+F 3 "" H 12050 6650 50  0001 C CNN
+	1    12050 6650
+	1    0    0    -1
+$EndComp
+$Comp
+L power:+3.3V #PWR0104
+U 1 1 5E87E8A2
+P 3150 8600
+F 0 "#PWR0104" H 3150 8450 50  0001 C CNN
+F 1 "+3.3V" H 3165 8773 50  0000 C CNN
+F 2 "" H 3150 8600 50  0001 C CNN
+F 3 "" H 3150 8600 50  0001 C CNN
+	1    3150 8600
+	1    0    0    -1
+$EndComp
+Text Label 1050 6450 0    50   ~ 0
+ME_A
+Text Label 1050 6550 0    50   ~ 0
+ME_B
+Wire Wire Line
+	1550 6450 1050 6450
+Wire Wire Line
+	1550 6550 1050 6550
 $EndSCHEMATC

Commit message: pcb rev 1-2
Connections:
- net +3V3: now also MODULE1.1 (Pin_1)
- net +5V: no longer MODULE1.1 (Pin_1)
Changed lines of the file:
@@
-	1    0    0    -1
-$EndComp
-$Comp
-L power:+5V #PWR033
-U 1 1 5EF8E422
-P 12400 1100
-F 0 "#PWR033" H 12400 950 50  0001 C CNN
-F 1 "+5V" H 12250 1150 50  0000 C CNN
-F 2 "" H 12400 1100 50  0001 C CNN
-F 3 "" H 12400 1100 50  0001 C CNN
-	1    12400 1100
 	1    0    0    -1
 $EndComp
@@
 Wire Wire Line
 	1550 6550 1050 6550
+$Comp
+L power:+3.3V #PWR?
+U 1 1 5E84D9E3
+P 12400 1100
+F 0 "#PWR?" H 12400 950 50  0001 C CNN
+F 1 "+3.3V" H 12415 1273 50  0000 C CNN
+F 2 "" H 12400 1100 50  0001 C CNN
+F 3 "" H 12400 1100 50  0001 C CNN
+	1    12400 1100
+	1    0    0    -1
+$EndComp
 $EndSCHEMATC
